File: eagle/main.brd (EAGLE design)
At the start: 64.5 x 52.8 mm, 66 parts, among them IC1 317EMP, IC2 74AHC1G125DCK, IC3 74AHC1G125DCK, U1 ESP-WROOM-32, U2 MCP2200, U3 MICROSD, U4 ATSAMD21G-A, Y1 12M

Commit message: rev4
Parts:
- added ATLED: 0805, led:SML0805
- added C14, C15: 18p, SparkFun-Capacitors:0603-CAP
- added J13: (no value), SparkFun-Connectors:1X04-1.27MM
- added R19: 303, SparkFun-Resistors:0805
- added Y2: 12M, SparkFun-FreqCtrl:CRYSTAL-TXC-7A
- moved D1 12.3 mm to (59.4, 36.1), turned to 180 degrees
- moved R18 2.02 mm to (53.7, 10.0)
- moved PWRLED 1.52 mm to (60.2, 44.7)
- moved R1 1.30 mm to (57.7, 44.2)
- moved C10 0.92 mm to (50.5, 13.2)
Connections:
- removed net IO27: J4.4, U1.12
- removed net VIN: D1.A, JP1.1, R18.2, USB1.VBUS
- new net ATCLK: J3.2, J4.3, U1.30, U4.45
- new net ATCS: J3.4, U1.28, U4.39
- new net ATIO: J4.4, U1.12, U4.46
- new net N$13: J13.1, U4.3
- new net N$14: J13.2, U4.4
- new net N$20: C15.1, U4.24, Y2.P$1
- new net N$34: C14.1, U4.23, Y2.P$2
- new net N$4: ATLED.A, R19.2
- new net N$8: J13.3, U4.2
- net 5V: now also JP1.1, R18.2, USB1.VBUS
- net GND: now also ATLED.C, C14.2, C15.2, D1.A; no longer J4.3
- net IO12: no longer U4.47
- net IO13: no longer U4.46
- net IO14: no longer U4.1
- net IO15: no longer U4.48
- net IO4: no longer U4.45
- net N$2: now also R19.1, U4.48; no longer J3.2, U1.30
- net N$5: now also R5.1
- net N$6: now also J13.4, U4.1; no longer J3.4, R5.1, U1.28
Routing:
- net ATCLK: track 0.00 -> 91.9 mm, vias 0 -> 2
- net ATCS: track 0.00 -> 68.4 mm
- net ATIO: track 0.00 -> 63.2 mm, vias 0 -> 2
- net IO14: track 73.3 -> 27.2 mm
- net IO15: track 75.7 -> 37.6 mm
- net IO12: track 62.1 -> 35.2 mm
- net IO27: track 26.2 -> 0.00 mm
- net 5V: track 71.5 -> 97.3 mm, vias 0 -> 1
- net IO13: track 59.1 -> 33.7 mm
- net VIN: track 21.6 -> 0.00 mm, vias 1 -> 0
- net N$6: track 29.0 -> 8.51 mm
- net N$2: track 21.7 -> 4.69 mm
- net GND: track 41.6 -> 57.1 mm
- net N$8: track 0.00 -> 8.08 mm
- net N$14: track 0.00 -> 7.65 mm
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Other:
- board text added: "ATIO"
- board text added: "ATLED"
- board text added: "PROG"
- board text added: "RESET"
- board text added: "rev 4"
- board text removed: "rev 3"
