File: eagle/main.sch (EAGLE design)
At the start: 65 parts, among them IC1 317EMP, IC2 74AHC1G125DCK, IC3 74AHC1G125DCK, Q1 MOSFET-NCHANNELBSS138, Q2 MOSFET-NCHANNELBSS138, Q3 MOSFET-NCHANNELBSS138, U1 ESP-WROOM-32, U2 MCP2200, U3 MICROSD, U4 ATSAMD21G-A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

Commit message: rev4
Parts:
- added ATLED: 0805, led:LEDSML0805
- added C14, C15: 18p, SparkFun-Capacitors:CAP0603-CAP
- added J13: (no value), SparkFun-Connectors:M041.27MM
- added R19: 303, SparkFun-Resistors:RESISTOR0805-RES
- added Y2: 12M, SparkFun-FreqCtrl:CRYSTALTXC-7A
Connections:
- removed net IO27: J4.4, U1.IO27
- removed net VIN: D1.A, JP1.1, R18.2, USB1.VBUS
- new net ATCLK: J3.2, J4.3, U1.IO18, U4.PA30(SWCLK/SER1:2+)
- new net ATCS: J3.4, U1.IO17, U4.PA27
- new net ATIO: J4.4, U1.IO27, U4.PA31(SWDIO/SER1:3+)
- new net N$13: J13.1, U4.PA02(AIN0/DAC)
- new net N$14: J13.2, U4.PA03(AIN1/REFA)
- new net N$20: C15.1, U4.PA15(XOUT/SER2:3+), Y2.1
- new net N$34: C14.1, U4.PA14(XIN/SER2:2+), Y2.2
- new net N$4: ATLED.A, R19.2
- new net N$8: J13.3, U4.PA01(XOUT32/SER1:1/TC2:1)
- net 5V: now also JP1.1, R18.2, USB1.VBUS
- net GND: now also ATLED.C, C14.2, C15.2, D1.A; no longer J4.3
- net IO12: no longer U4.PB02(AIN10/SER5:0)
- net IO13: no longer U4.PA31(SWDIO/SER1:3+)
- net IO14: no longer U4.PA00(XIN32/SER1:0/TC2:0)
- net IO15: no longer U4.PB03(AIN11/SER5:1)
- net IO4: no longer U4.PA30(SWCLK/SER1:2+)
- net N$2: now also R19.1, U4.PB03(AIN11/SER5:1); no longer J3.2, U1.IO18
- net N$5: now also R5.1
- net N$6: now also J13.4, U4.PA00(XIN32/SER1:0/TC2:0); no longer J3.4, R5.1, U1.IO17
Other:
- moved on the sheet: D1
